File: placainterruptores.sch (KiCad schematic (older format))
At the start: 66 parts, among them J1 USB, P1 CONN_2, P10 CONN_2, P11 CONN_2, P12 CONN_2, P13 CONN_2, P14 CONN_2, P15 CONN_2, P16 CONN_2, P17 CONN_2, P2 CONN_2, P3 CONN_2, P4 CONN_2, P5 CONN_2, P6 CONN_2, P7 CONN_2, P8 CONN_2, P9 CONN_2, Q1 BC547, Q2 BC547, Q3 BC547, Q4 BC547, Q5 BC547, Q6 BC547, Q7 BC547, Q8 BC547, SW1 3WAY_SWITCH, SW2 3WAY_SWITCH, SW3 3WAY_SWITCH, SW4 3WAY_SWITCH, SW5 3WAY_SWITCH, SW6 3WAY_SWITCH, SW7 3WAY_SWITCH, SW8 3WAY_SWITCH

Commit message: Ahora no hay que pasar por HiZ para ir desde 5V a GND, lo que mejora la generación de flancos de subida/bajada. Placa adaptada para la nueva versión de Kicad. Nuevos ficheros de fabricación generados
Parts:
- added D9: DIODE, Discret:D3, symbol DIODE
- D1, D2, D3, D4, D5, D6, D7, D8: footprint LED-0805 -> LEDs:LED-0805
- J1: footprint USB_MINI_B -> Connect:USB_MINI_B
- P1: footprint 2PIN_6mm -> Divers:2PIN_6mm
- P10, P11, P12, P13, P14, P15, P16, P17, P2, P3, P4, P5, P6, P7, P8, P9: footprint SIL-2 -> Connect:SIL-2
- Q1, Q2, Q3, Q4, Q5, Q6, Q7, Q8: footprint TO92 -> Discret:TO92-123
- R1, R10, R11, R12, R13, R14, R15, R16, R17, R18, R19, R2, R20, R21, R22, R23, R24, R3, R4, R5, R6, R7, R8, R9: footprint SM0805 -> Resistors_SMD:R_0805
- SW1, SW2, SW3, SW4, SW5, SW6, SW7, SW8: footprint 3WAY-SWITCH -> PI2:3WAY-SWITCH
Connections:
- net +5V: now also D9.2 (K)
- net GND: now also D9.1 (A)
- net at R17.2: now also SW1.3; no longer SW1.1
- net at R18.2: now also SW2.3; no longer SW2.1
- net at R19.2: now also SW3.3; no longer SW3.1
- net at R20.2: now also SW4.3; no longer SW4.1
- net at R21.2: now also SW5.3; no longer SW5.1
- net at R22.2: now also SW6.3; no longer SW6.1
- net at R23.2: now also SW7.3; no longer SW7.1
- net at R24.2: now also SW8.3; no longer SW8.1
Other:
- moved on the sheet: R17, R18, R19, R20, R21, R22, R23, R24
